Commit message: 新增urdf joint constrain

File: urdf/big_red_dog.urdf (robot description, URDF)
Before this commit: robot big_red_dog, 35 links, 34 joints
Joints:
- joint FL_calf_joint: limit lower=0 upper=0 effort=0 velocity=0 -> lower=-3.14 upper=3.14 effort=0 velocity=0
- joint FL_hip_joint: limit lower=0 upper=0 effort=0 velocity=0 -> lower=-0.61 upper=0.61 effort=0 velocity=0
- joint FL_thigh_joint: limit lower=0 upper=0 effort=0 velocity=0 -> lower=-1.5708 upper=1.5708 effort=0 velocity=0
- joint FR_calf_joint: limit lower=0 upper=0 effort=0 velocity=0 -> lower=-3.14 upper=3.14 effort=0 velocity=0
- joint FR_hip_joint: limit lower=0 upper=0 effort=0 velocity=0 -> lower=-0.61 upper=0.61 effort=0 velocity=0
- joint FR_thigh_joint: limit lower=0 upper=0 effort=0 velocity=0 -> lower=-1.5708 upper=1.5708 effort=0 velocity=0
- joint RL_calf_joint: limit lower=0 upper=0 effort=0 velocity=0 -> lower=-3.14 upper=3.14 effort=0 velocity=0
- joint RL_hip_joint: limit lower=0 upper=0 effort=0 velocity=0 -> lower=-0.61 upper=0.61 effort=0 velocity=0
- joint RL_thigh_joint: limit lower=0 upper=0 effort=0 velocity=0 -> lower=-1.5708 upper=1.5708 effort=0 velocity=0
- joint RR_calf_joint: limit lower=0 upper=0 effort=0 velocity=0 -> lower=-3.14 upper=3.14 effort=0 velocity=0
- joint RR_hip_joint: limit lower=0 upper=0 effort=0 velocity=0 -> lower=-0.61 upper=0.61 effort=0 velocity=0
- joint RR_thigh_joint: limit lower=0 upper=0 effort=0 velocity=0 -> lower=-1.5708 upper=1.5708 effort=0 velocity=0

Commit message: 更改joint方向

File: urdf/big_red_dog.urdf (robot description, URDF)
Before this commit: robot big_red_dog, 35 links, 34 joints
Joints:
- joint FL_calf_joint: axis 0 -1 0 -> 0 1 0
- joint FL_hip_joint: axis -1 0 0 -> 1 0 0
- joint FL_thigh_joint: axis 0 -1 0 -> 0 1 0
- joint FR_hip_joint: axis -1 0 0 -> 1 0 0
- joint RL_calf_joint: axis 0 -1 0 -> 0 1 0
- joint RL_thigh_joint: axis 0 -1 0 -> 0 1 0
